File: proto/sensorBoard.brd (EAGLE design)
At the start: 160 x 100 mm, 4 parts, among them U1 BME280, U5 ATMEGA328P_TQFP

Commit message: PCB
Parts:
- removed BT1: (no value), SparkFun-Batteries:BATTCOM_20MM_PTH
- removed U5: ATMEGA328P_TQFP, SparkFun-IC-Microcontroller:TQFP32-08
- added C1: 0,47u, PDI_PassiveComponents:C0805K
- added C2: 22u, PDI_PassiveComponents:C0805K
- added C3: 100u, PDI_PassiveComponents:CAPAE660X800
- added C4, C5: 0,1u, PDI_PassiveComponents:C0805K
- added IC1: TS2940SOT223, PDI_Semiconductors:SOT230P700X180-4
- added J1: MICRO-USB, PDI_Connectors:MOLEX_105017-0001
- added J2: CONN-2X3MALE, PDI_Connectors:HDRV6W64P254_2X3_762X508X838B
- added LED1: (no value), PDI_Semiconductors:LED0805
- added R1: 4,7k, PDI_PassiveComponents:R0805
- added R2: 33, PDI_PassiveComponents:R0805
- added R3: 100, PDI_PassiveComponents:R0805
- added R4: 10k, PDI_PassiveComponents:R0805
- added SW1: SWITCH, PDI_MechanicalComponents:EG1215AA
- added U$1: ATTINY3217TQFN-24, PDI_Semiconductors:QFN50P400X400X80-25T270
- added U$3: CR24773039, PDI_MechanicalComponents:CR2477
- U1: device BME280:PSON65P250X250X100-8N -> PDI_Semiconductors:PSON65P250X250X100-8N
- moved SV1 72.2 mm to (14.0, 2.54), turned to 180 degrees
Connections:
- removed net +: BT1.1
- removed net +3.3V: U1.8
- removed net -: BT1.2
- removed net VDDIO: U1.6
- new net +3V3: C3.1, C4.1, C5.1, J2.2, R2.2, R4.1, SV1.1, U$1.4, U1.2, U1.6, U1.8
- new net BT_ACT: SV1.5, U$1.7
- new net BT_RDY: SV1.6, U$1.6
- new net BT_REQ: SV1.7, U$1.5
- new net BT_RST: SV1.4, U$1.8
- new net MISO: J2.1, SV1.9, U$1.1
- new net MOSI: J2.4, SV1.8, U$1.24
- new net N$1: R1.1, SW1.1
- new net N$2: C1.1, IC1.1, J1.1
- new net N$3: C2.1, IC1.3, R3.1, SW1.3
- new net N$4: R1.2, U$3.P$1, U$3.P$2
- new net N$5: R2.1, SW1.2
- new net N$7: C3.2
- new net N$8: LED1.A, R3.2
- new net RST: J2.5, R4.2, U$1.23
- new net SCK: J2.3, SV1.10, U$1.2
- new net SCL: U$1.16, U1.4
- new net SDA: U$1.15, U1.3
- net GND: now also C1.2, C2.2, C4.2, C5.2, IC1.2, IC1.4, J1.5, J2.6, LED1.K, SV1.2, U$1.25, U$1.3, U$3.P$3, U1.5; no longer U5.21, U5.3, U5.5
Other:
- board size 160 x 100 mm -> 27.9 x 29.2 mm
