File: proto/sensorBoard.sch (EAGLE design)
At the start: 4 parts, among them U1 BME280, U5 ATMEGA328P_TQFP

Commit message: PCB
Parts:
- removed BT1: (no value), SparkFun-Batteries:BATTERY-20MM_PTH
- removed U5: ATMEGA328P_TQFP, SparkFun-IC-Microcontroller:ATMEGA328P_TQFP
- added C1: 0,47u, PDI_PassiveComponents:SMD-CAPACITORC0805
- added C2: 22u, PDI_PassiveComponents:SMD-CAPACITORC0805
- added C3: 100u, PDI_PassiveComponents:SMD-ELECTROLYTIC-CAPACITORD8
- added C4, C5: 0,1u, PDI_PassiveComponents:SMD-CAPACITORC0805
- added IC1: TS2940SOT223, PDI_Semiconductors:TS2940SOT223
- added J1: MICRO-USB, PDI_Connectors:MICRO-USB
- added J2: CONN-2X3MALE, PDI_Connectors:CONN-2X3MALE
- added LED1: (no value), PDI_Semiconductors:LED0805
- added R1: 4,7k, PDI_PassiveComponents:SMD-RESISTORR0805
- added R2: 33, PDI_PassiveComponents:SMD-RESISTORR0805
- added R3: 100, PDI_PassiveComponents:SMD-RESISTORR0805
- added R4: 10k, PDI_PassiveComponents:SMD-RESISTORR0805
- added SW1: SWITCH, PDI_MechanicalComponents:SWITCH
- added U$1: ATTINY3217TQFN-24, PDI_Semiconductors:ATTINY3217TQFN-24
- added U$3: CR24773039, PDI_MechanicalComponents:CR24773039
- U1: device BME280:BME280 -> PDI_Semiconductors:BME280
Connections:
- new net +3V3: C3.+, C4.1, C5.1, J2.2, R2.2, R4.1, SV1.1, U$1.VCC, U1.CSB, U1.VDD, U1.VDDIO
- new net BT_ACT: SV1.5, U$1.PA6
- new net BT_RDY: SV1.6, U$1.PA5
- new net BT_REQ: SV1.7, U$1.PA4/!SS!
- new net BT_RST: SV1.4, U$1.PA7
- new net MISO: J2.1, SV1.9, U$1.PA2/MISO
- new net MOSI: J2.4, SV1.8, U$1.PA1/MOSI
- new net N$1: R1.1, SW1.NC
- new net N$2: C1.1, IC1.IN, J1.VDD
- new net N$3: C2.1, IC1.OUT, R3.1, SW1.NO
- new net N$4: R1.2, U$3.P
- new net N$5: R2.1, SW1.COM
- new net N$7: C3.-
- new net N$8: LED1.A, R3.2
- new net RST: J2.5, R4.2, U$1.PA0/!RESET!/UPDI
- new net SCK: J2.3, SV1.10, U$1.PA3/EXTCLK/SCK
- new net SCL: U$1.PB0/SCL, U1.SCK
- new net SDA: U$1.PB1/SDA, U1.SDI
- net GND: now also C1.2, C2.2, C4.2, C5.2, IC1.GND, J1.GND, J2.6, LED1.C, SV1.2, U$1.EPAD, U$1.GND, U$3.N, U1.SDO; no longer U5.AGND, U5.GND@3, U5.GND@5
Other:
- moved on the sheet: SV1
